File: hardware/cube3.kicad_pcb (KiCad board)
At the start: 2 copper layers, 43 parts, among them K0 RGB_CATHODE, K1 RGB_CATHODE, K8 RGB_CATHODE, K9 RGB_CATHODE, P1 POWER, P10 C_IN, P11 CONN_1, P12 CONN_1, P13 CONN_1, P14 CONN_1, P15 A1, P2 POWER, P3 DATA_IN, P4 DATA_OUT, P5 ISP, P6 A0, P7 A0, P8 A1, P9 C_OUT, Q1 AP4435GH, Q2 AP4435GH, Q3 CONN_3, Q4 CONN_3, SW1 RESET, U1 TLC5940, U2 TLC5940, U3 TLC5940, U4 ATMEGA328, X1 16MHz

Commit message: Final hardware tweaks.
Signed-off-by: Paul Brook <paul@nowt.org>
Parts:
- added R7: 0, SM0603, B.Cu at (109.9, 81.9)
- added R8: 0, SM0603, B.Cu at (107.3, 81.9)
- P10: value C_IN -> K_IN
- P3: value DATA_IN -> DATA
- P4: value DATA_OUT -> DATA
- P9: value C_OUT -> K_OUT
- R5: footprint R4-LARGE_PADS -> R3-5
- moved R5 0.64 mm to (109.2, 73.7)
Connections:
- U4 pad 12: /BLANK -> /GSCK
- U4 pad 13: /DCPRG -> /BLANK
- U4 pad 14: /GSCK -> /DCPRG
- U4 pad 25: (no net) -> /VPRG
- U4 pad 26: /VPRG -> (no net)
- U4 pad 27: (no net) -> /ID0
- U4 pad 28: (no net) -> /ID1
Routing:
- net /5v: track 311.5 -> 322.0 mm
- net /GSCK: track 113.9 -> 109.2 mm, vias 1 -> 2
- net /ID1: track 0.00 -> 2.68 mm
- net /ID0: track 0.00 -> 2.68 mm
- net /BLANK: track 119.7 -> 117.2 mm
- net /r1: track 96.9 -> 99.1 mm
- net /GND: vias 5 -> 6
Other:
- board text added: "(SYNCA) (SYNCB) SCK MOSI CS GND"
- board text added: "0"
- board text added: "1"
- board text added: "B0"
- board text added: "B10"
- board text added: "B13"
- board text added: "B15"
- board text added: "B2"
- board text added: "B5"
- board text added: "B7"
- board text added: "B8"
- board text added: "G0"
- board text added: "G10"
- board text added: "G13"
- board text added: "G15"
- board text added: "G2"
- board text added: "G5"
- board text added: "G7"
- board text added: "G8"
- board text added: "ID"
- board text added: "R0"
- board text added: "R1"
- board text added: "R10"
- board text added: "R13"
- board text added: "R15"
- board text added: "R5"
- board text added: "R7"
- board text added: "R8"
